File: luckybamboo/luckybamboo.sch (KiCad schematic (older format))
At the start: 148 parts, among them J1 NEIGHBOR1, J10 TEST_2P, J11 TEST_2P, J12 TEST_2P, J13 TEST_2P, J14 TEST_2P, J15 TEST_2P, J16 TEST_2P, J17 Conn_Coaxial, J18 Conn_Coaxial, J19 TEST_2P, J2 NEIGHBOR2, J20 TEST_2P, J21 TEST_2P, J22 TEST_2P, J23 TEST_2P, J24 TEST_2P, J25 TEST_2P, J26 TEST_2P, J27 TEST_2P, J28 TEST_2P, J29 TEST_2P, J3 Conn_01x08, J30 TEST_2P, J31 TEST_2P, J32 TEST_2P, J33 TEST_2P, J4 Conn_01x08, J5 Conn_01x08, J6 Conn_01x08, J7 BONUS_ROW, J8 TEST_2P, J9 TEST_2P, U1 ADF7242, U10 ADF7242_balun, U11 ADF7242_balun, U12 HHM2293A1, U13 BGA7H1N6, U14 ADF7242_balun, U15 ADF7242_balun, U16 ADF7242_balun, U17 ADF7242_balun, U2 ADF7242, U3 ADF7242, U4 ADF7242, U5 SKY13322, U6 HHM2293A1, U7 HHM2293A1, U8 ADF7242_balun, U9 ADF7242_balun, X1 XTAL4PIN, X2 XTAL4PIN, X3 XTAL4PIN, X4 XTAL4PIN

Commit message: BOM: Changed SMA connectors to RP-SMA and changed SPORT header
Parts:
- J17: Description CONN SMA RCPT STR 50OHM EDGE MNT -> CONN RPSMA PLG STR 50OHM EDGEMNT; Part Number CONSMA003.062 -> CONREVSMA013.062
- J3, J4, J5, J6: Description CONN RECEPT 2MM DUAL STR 8POS -> CONN RCPT 8POS 0.1 GOLD PCB; Manufacturer Sullins Connector Solutions -> Samtec Inc.; Part Number NPPN042AFCN-RC -> CES-104-01-L-D
- U12, U6, U7: symbol gsg-symbols:HHM2293A1 -> luckybamboo-rescue:HHM2293A1-gsg-symbols
- U13: symbol gsg-symbols:BGA7H1N6 -> luckybamboo-rescue:BGA7H1N6-gsg-symbols
Changed lines of the file:
@@
 F 2 "gsg-modules:SMA-EDGE" H 10150 2100 50  0001 C CNN
 F 3 "" H 10150 2100 50  0001 C CNN
-F 4 " CONN SMA RCPT STR 50OHM EDGE MNT" H 10160 2320 50  0001 C CNN "Description"
+F 4 " CONN RPSMA PLG STR 50OHM EDGEMNT" H 10160 2320 50  0001 C CNN "Description"
 F 5 "Linx Technologies Inc." H 10160 2320 50  0001 C CNN "Manufacturer"
-F 6 "CONSMA003.062" H 10160 2320 50  0001 C CNN "Part Number"
+F 6 "CONREVSMA013.062" H 10160 2320 50  0001 C CNN "Part Number"
 	1    10150 2100
 	-1   0    0    1
@@
 F 2 "gsg-modules:HEADER-2x4" H 4850 950 50  0001 C CNN
 F 3 "" H 4850 950 50  0001 C CNN
-F 4 " CONN RECEPT 2MM DUAL STR 8POS" H 4850 1450 50  0001 C CNN "Description"
-F 5 "Sullins Connector Solutions" H 4850 1450 50  0001 C CNN "Manufacturer"
-F 6 "NPPN042AFCN-RC" H 4850 1450 50  0001 C CNN "Part Number"
+F 4 "CONN RCPT 8POS 0.1 GOLD PCB" H 4850 1450 50  0001 C CNN "Description"
+F 5 "Samtec Inc." H 4850 1450 50  0001 C CNN "Manufacturer"
+F 6 "CES-104-01-L-D" H 4850 1450 50  0001 C CNN "Part Number"
 	1    4850 950
 	1    0    0    -1
@@
 F 2 "gsg-modules:HEADER-2x4" H 9650 950 50  0001 C CNN
 F 3 "" H 9650 950 50  0001 C CNN
-F 4 " CONN RECEPT 2MM DUAL STR 8POS" H 9650 1450 50  0001 C CNN "Description"
-F 5 "Sullins Connector Solutions" H 9650 1450 50  0001 C CNN "Manufacturer"
-F 6 "NPPN042AFCN-RC" H 9650 1450 50  0001 C CNN "Part Number"
+F 4 "CONN RCPT 8POS 0.1 GOLD PCB" H 9650 1450 50  0001 C CNN "Description"
+F 5 "Samtec Inc." H 9650 1450 50  0001 C CNN "Manufacturer"
+F 6 "CES-104-01-L-D" H 9650 1450 50  0001 C CNN "Part Number"
 	1    9650 950
 	1    0    0    -1
@@
 F 2 "gsg-modules:HEADER-2x4" H 5050 5800 50  0001 C CNN
 F 3 "" H 5050 5800 50  0001 C CNN
-F 4 " CONN RECEPT 2MM DUAL STR 8POS" H 5050 6300 50  0001 C CNN "Description"
-F 5 "Sullins Connector Solutions" H 5050 6300 50  0001 C CNN "Manufacturer"
-F 6 "NPPN042AFCN-RC" H 5050 6300 50  0001 C CNN "Part Number"
+F 4 "CONN RCPT 8POS 0.1 GOLD PCB" H 5050 6300 50  0001 C CNN "Description"
+F 5 "Samtec Inc. " H 5050 6300 50  0001 C CNN "Manufacturer"
+F 6 "CES-104-01-L-D" H 5050 6300 50  0001 C CNN "Part Number"
 	1    5050 5800
 	1    0    0    -1
@@
 $EndComp
 $Comp
-L gsg-symbols:HHM2293A1 U7
+L luckybamboo-rescue:HHM2293A1-gsg-symbols U7
 U 1 1 5BDFC016
 P 10250 7900
@@
 	9700 7700 9650 7700
 $Comp
-L gsg-symbols:HHM2293A1 U6
+L luckybamboo-rescue:HHM2293A1-gsg-symbols U6
 U 1 1 5BDFC052
 P 10250 9400
@@
 	9650 9200 9350 9200
 $Comp
-L gsg-symbols:BGA7H1N6 U13
+L luckybamboo-rescue:BGA7H1N6-gsg-symbols U13
 U 1 1 5BDFBFD4
 P 12800 7450
@@
 F 2 "gsg-modules:HEADER-2x4" H 9700 5800 50  0001 C CNN
 F 3 "" H 9700 5800 50  0001 C CNN
-F 4 " CONN RECEPT 2MM DUAL STR 8POS" H 9700 6300 50  0001 C CNN "Description"
-F 5 "Sullins Connector Solutions" H 9700 6300 50  0001 C CNN "Manufacturer"
-F 6 "NPPN042AFCN-RC" H 9700 6300 50  0001 C CNN "Part Number"
+F 4 "CONN RCPT 8POS 0.1 GOLD PCB" H 9700 6300 50  0001 C CNN "Description"
+F 5 "Samtec Inc." H 9700 6300 50  0001 C CNN "Manufacturer"
+F 6 "CES-104-01-L-D" H 9700 6300 50  0001 C CNN "Part Number"
 	1    9700 5800
 	1    0    0    -1
@@
 RFIN2
 $Comp
-L gsg-symbols:HHM2293A1 U12
+L luckybamboo-rescue:HHM2293A1-gsg-symbols U12
 U 1 1 5BDFBFCD
 P 11900 8750

Commit message: Changed  Changed SPI CS 3 and IRQ1 3 pins, which were interfering with SPIFI. Added DC blocking capacitors near TX switch
Parts:
- added C62, C66, C67, C82, C83: 47pF, gsg-modules:0402, symbol luckybamboo-rescue:C
- U1, U2, U3, U4: symbol luckybamboo-rescue:ADF7242 -> gsg-symbols:ADF7242
- U10, U11, U14, U15, U16, U17, U8, U9: symbol luckybamboo-rescue:ADF7242_balun -> gsg-symbols:ADF7242_balun
- U12, U6, U7: symbol luckybamboo-rescue:HHM2293A1-gsg-symbols -> gsg-symbols:HHM2293A1
- U13: symbol luckybamboo-rescue:BGA7H1N6-gsg-symbols -> gsg-symbols:BGA7H1N6
- U5: symbol luckybamboo-rescue:SKY13322 -> gsg-symbols:SKY13322
Connections:
- wire segments 511 -> 520
Other:
- moved on the sheet: J18
