File: luckybamboo/luckybamboo.sch (KiCad schematic (older format))
At the start: 153 parts, among them J1 NEIGHBOR1, J10 TEST_2P, J11 TEST_2P, J12 TEST_2P, J13 TEST_2P, J14 TEST_2P, J15 TEST_2P, J16 TEST_2P, J17 Conn_Coaxial, J18 Conn_Coaxial, J19 TEST_2P, J2 NEIGHBOR2, J20 TEST_2P, J21 TEST_2P, J22 TEST_2P, J23 TEST_2P, J24 TEST_2P, J25 TEST_2P, J26 TEST_2P, J27 TEST_2P, J28 TEST_2P, J29 TEST_2P, J3 Conn_01x08, J30 TEST_2P, J31 TEST_2P, J32 TEST_2P, J33 TEST_2P, J4 Conn_01x08, J5 Conn_01x08, J6 Conn_01x08, J7 BONUS_ROW, J8 TEST_2P, J9 TEST_2P, U1 ADF7242, U10 ADF7242_balun, U11 ADF7242_balun, U12 HHM2293A1, U13 BGA7H1N6, U14 ADF7242_balun, U15 ADF7242_balun, U16 ADF7242_balun, U17 ADF7242_balun, U2 ADF7242, U3 ADF7242, U4 ADF7242, U5 SKY13322, U6 HHM2293A1, U7 HHM2293A1, U8 ADF7242_balun, U9 ADF7242_balun, X1 XTAL4PIN, X2 XTAL4PIN, X3 XTAL4PIN, X4 XTAL4PIN

Commit message: Lucky Bamboo: Rerouted RX RF signals and rearranged schematic to be consistent with layout. Gladiolus: Routed incomplete signal near TX transistor.
Parts:
- J17: Description CONN RPSMA PLG STR 50OHM EDGEMNT -> CONN RPSMA PLG STR 50OHM EDGEMNT
- J18: Description CONN SMA RCPT STR 50OHM EDGE MNT -> CONN RPSMA PLG STR 50OHM EDGEMNT; Part Number CONSMA003.062 -> CONREVSMA013.062
Connections:
- net RFIN1: now also R10.1, U7.3 (RFOUT2); no longer R9.2, U6.1 (RFOUT1)
- net RFIN2: now also R9.2, U6.1 (RFOUT1); no longer R9.1, U6.3 (RFOUT2)
- net RFIN4: now also R9.1, U6.3 (RFOUT2); no longer R10.1, U7.3 (RFOUT2)
Other:
- moved on the sheet: C12, C13, C14, C18, C19, C2, C20, C22, C25, C26, C29, C30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

Commit message: Replaced rescued symbols on Gladiolus and Lucky Bamboo. Lucky Bamboo: Shorted IRQ1/IRQ2 jumpers to create default connections.
Parts:
- C1, C10, C11, C12, C13, C14, C15, C16, C17, C18, C19, C2, C20, C21, C22, C23, C24, C25, C26, C27, C28, C29, C3, C30, C31, C32, C33, C34, C35, C36, C37, C38, C39, C4, C40, C41, C42, C43, C44, C45, C46, C47, C48, C49, C5, C50, C51, C52, C53, C54, C55, C56, C57, C58, C59, C6, C60, C61, C62, C63, C64, C65, C66, C67, C68, C69, C7, C70, C71, C72, C73, C74, C75, C76, C77, C78, C79, C8, C80, C81, C82, C83, C9: symbol luckybamboo-rescue:C -> Device:C
- J1, J2: symbol luckybamboo-rescue:CONN_02X20 -> Connector_Generic:Conn_02x20_Odd_Even
- J17, J18: symbol luckybamboo-rescue:Conn_Coaxial -> Connector:Conn_Coaxial
- J3, J4, J5, J6: symbol luckybamboo-rescue:Conn_01x08 -> Connector_Generic:Conn_01x08
- L1: symbol luckybamboo-rescue:L -> Device:L
- R1, R10, R11, R2, R3, R4, R5, R6, R7, R8, R9: symbol luckybamboo-rescue:R -> Device:R
- X1, X2, X3, X4: symbol luckybamboo-rescue:XTAL4PIN -> gsg-symbols:XTAL4PIN
Connections:
- net P1_0 is gone; now on net DR2: J1.7 (Pin_7), J11.2
- net P1_16 is gone; now on net DR4: J1.30 (Pin_30), J15.2
- net P2_2 is gone; now on net DR3: J13.2, J2.33 (Pin_33)
- net P6_3 is gone; now on net DR1: J2.36 (Pin_36), J9.2
- net ~CS~1 is gone; now on net P4_3: J19.1, J20.1, R3.2, U1.24 (~CS~)
- net ~CS~2 is gone; now on net P5_2: J21.1, J22.1, R7.2, U2.24 (~CS~)
- net ~CS~3 is gone; now on net P6_7: J23.1, J24.1, R4.2, U3.24 (~CS~)
- net ~CS~4 is gone; now on net P9_6: J25.1, J26.1, R8.2, U4.24 (~CS~)
Other:
- moved on the sheet: J17, J18
